File: splyd.kicad_pcb (KiCad board)
At the start: 2 copper layers, 156.2 x 146.6 mm, 74 parts, among them J0 AudioJack3, J1 USB from Pro micro, K00 KEYSW, K01 KEYSW, K02 KEYSW, K03 KEYSW, K04 KEYSW, K05 KEYSW, K10 KEYSW, K11 KEYSW, K12 KEYSW, K13 KEYSW, K14 KEYSW, K15 KEYSW, K16 KEYSW, K20 KEYSW, K21 KEYSW, K22 KEYSW, K23 KEYSW, K24 KEYSW, K25 KEYSW, K26 KEYSW, K30 KEYSW, K31 KEYSW, K32 KEYSW, K33 KEYSW, K34 KEYSW, K35 KEYSW, K36 KEYSW, K43 KEYSW, K44 KEYSW, K45 KEYSW, K46 KEYSW, K54 KEYSW, K55 KEYSW, K56 KEYSW, U0 Pro Micro

Commit message: Add right hand and prepare footprint placements
Parts:
- removed USB1: USB C receptacle, Type-C:USB_C_GCT_USB4085
- added DR1: D, keyboard_parts:D_SOD123_axial, B.Cu at (238.2, 69.5)
- added DR10: D, keyboard_parts:D_SOD123_axial, B.Cu at (219.1, 90.5)
- added DR11: D, keyboard_parts:D_SOD123_axial, B.Cu at (238.2, 88.6)
- added DR12: D, keyboard_parts:D_SOD123_axial, B.Cu at (257.2, 83.8)
- added DR13: D, keyboard_parts:D_SOD123_axial, B.Cu at (276.2, 76.2)
- added DR14: D, keyboard_parts:D_SOD123_axial, B.Cu at (295.3, 84.7)
- added DR15: D, keyboard_parts:D_SOD123_axial, B.Cu at (314.4, 103.8)
- added DR16: D, keyboard_parts:D_SOD123_axial, B.Cu at (333.4, 107.6)
- added DR2: D, keyboard_parts:D_SOD123_axial, B.Cu at (257.2, 64.7)
- added DR20: D, keyboard_parts:D_SOD123_axial, B.Cu at (219.1, 109.5)
- added DR21: D, keyboard_parts:D_SOD123_axial, B.Cu at (238.2, 107.6)
- added DR22: D, keyboard_parts:D_SOD123_axial, B.Cu at (257.2, 102.8)
- added DR23: D, keyboard_parts:D_SOD123_axial, B.Cu at (276.2, 95.2)
- added DR24: D, keyboard_parts:D_SOD123_axial, B.Cu at (295.3, 103.8)
- added DR25: D, keyboard_parts:D_SOD123_axial, B.Cu at (314.4, 122.8)
- added DR26: D, keyboard_parts:D_SOD123_axial, B.Cu at (333.4, 126.7)
- added DR3: D, keyboard_parts:D_SOD123_axial, B.Cu at (276.2, 57.1)
- added DR30: D, keyboard_parts:D_SOD123_axial, B.Cu at (219.1, 128.6)
- added DR31: D, keyboard_parts:D_SOD123_axial, B.Cu at (238.2, 126.7)
- added DR32: D, keyboard_parts:D_SOD123_axial, B.Cu at (257.2, 121.9)
- added DR33: D, keyboard_parts:D_SOD123_axial, B.Cu at (276.2, 114.3)
- added DR34: D, keyboard_parts:D_SOD123_axial, B.Cu at (295.3, 122.8)
- added DR35: D, keyboard_parts:D_SOD123_axial, B.Cu at (314.4, 141.9)
- added DR36: D, keyboard_parts:D_SOD123_axial, B.Cu at (333.4, 145.7)
- added DR4: D, keyboard_parts:D_SOD123_axial, B.Cu at (295.3, 65.7)
- added DR40: D, keyboard_parts:D_SOD123_axial, B.Cu at (209.6, 156.2)
- added DR41: D, keyboard_parts:D_SOD123_axial, B.Cu at (219.1, 151.6)
- added DR42: D, keyboard_parts:D_SOD123_axial, B.Cu at (238.2, 151.4)
- added DR43: D, keyboard_parts:D_SOD123_axial, B.Cu at (257.2, 151.4)
- added DR5: D, keyboard_parts:D_SOD123_axial, B.Cu at (314.4, 84.7)
- added DR50: D, keyboard_parts:D_SOD123_axial, B.Cu at (218.1, 170.5)
- added DR51: D, keyboard_parts:D_SOD123_axial, B.Cu at (237.2, 170.5)
- added DR52: D, keyboard_parts:D_SOD123_axial, B.Cu at (256.2, 170.5)
- added DR6: D, keyboard_parts:D_SOD123_axial, B.Cu at (333.4, 88.6)
- added JR0: AudioJack3, mod_conn_av:jack_3.5_pj313d-smt, B.Cu at (316.3, 61.9)
- added JR1: USB from Pro micro, Connector_Wire:Pad_1x04_SMD_1x2mm, B.Cu at (322.9, 166.7)
- added KR01: KEYSW, keyswitches:Kailh_socket_MX, F.Cu at (238.2, 60.9)
- added KR02: KEYSW, keyswitches:Kailh_socket_MX, F.Cu at (257.2, 56.2)
- added KR03: KEYSW, keyswitches:Kailh_socket_MX, F.Cu at (276.2, 48.6)
- added KR04: KEYSW, keyswitches:Kailh_socket_MX, F.Cu at (295.3, 57.1)
- added KR05: KEYSW, keyswitches:Kailh_socket_MX, F.Cu at (314.4, 76.2)
- added KR06: KEYSW, keyswitches:Kailh_socket_MX, F.Cu at (333.4, 80.0)
- added KR10: KEYSW, keyswitches:Kailh_socket_MX, F.Cu at (219.1, 81.9)
- added KR11: KEYSW, keyswitches:Kailh_socket_MX, F.Cu at (238.2, 80.0)
- added KR12: KEYSW, keyswitches:Kailh_socket_MX, F.Cu at (257.2, 75.2)
- added KR13: KEYSW, keyswitches:Kailh_socket_MX, F.Cu at (276.2, 67.6)
- added KR14: KEYSW, keyswitches:Kailh_socket_MX, F.Cu at (295.3, 76.2)
- added KR15: KEYSW, keyswitches:Kailh_socket_MX, F.Cu at (314.4, 95.2)
- added KR16: KEYSW, keyswitches:Kailh_socket_MX, F.Cu at (333.4, 99.0)
- added KR20: KEYSW, keyswitches:Kailh_socket_MX, F.Cu at (219.1, 100.9)
- added KR21: KEYSW, keyswitches:Kailh_socket_MX, F.Cu at (238.2, 99.0)
- added KR22: KEYSW, keyswitches:Kailh_socket_MX, F.Cu at (257.2, 94.3)
- added KR23: KEYSW, keyswitches:Kailh_socket_MX, F.Cu at (276.2, 86.7)
- added KR24: KEYSW, keyswitches:Kailh_socket_MX, F.Cu at (295.3, 95.2)
- added KR25: KEYSW, keyswitches:Kailh_socket_MX, F.Cu at (314.4, 114.3)
- added KR26: KEYSW, keyswitches:Kailh_socket_MX, F.Cu at (333.4, 118.1)
- added KR30: KEYSW, keyswitches:Kailh_socket_MX, F.Cu at (219.1, 120.0)
- added KR31: KEYSW, keyswitches:Kailh_socket_MX, F.Cu at (238.2, 118.1)
- added KR32: KEYSW, keyswitches:Kailh_socket_MX, F.Cu at (257.2, 113.3)
- added KR33: KEYSW, keyswitches:Kailh_socket_MX, F.Cu at (276.2, 105.7)
- added KR34: KEYSW, keyswitches:Kailh_socket_MX, F.Cu at (295.3, 114.3)
- added KR35: KEYSW, keyswitches:Kailh_socket_MX, F.Cu at (314.4, 133.3)
- added KR36: KEYSW, keyswitches:Kailh_socket_MX, F.Cu at (333.4, 137.1)
- added KR40: KEYSW, keyswitches:Kailh_socket_MX, F.Cu at (209.6, 147.6)
- added KR41: KEYSW, keyswitches:Kailh_socket_MX, F.Cu at (228.6, 147.6)
- added KR42: KEYSW, keyswitches:Kailh_socket_MX, F.Cu at (247.7, 147.6)
- added KR43: KEYSW, keyswitches:Kailh_socket_MX, F.Cu at (266.7, 147.6)
- added KR50: KEYSW, keyswitches:Kailh_socket_MX, F.Cu at (209.6, 166.7)
- added KR51: KEYSW, keyswitches:Kailh_socket_MX, F.Cu at (228.6, 166.7)
- added KR52: KEYSW, keyswitches:Kailh_socket_MX, F.Cu at (247.7, 166.7)
- added RR0: 5.1K, Resistor_SMD:R_0603_1608Metric, B.Cu at (327.7, 69.7)
- added RR1: 5.1K, Resistor_SMD:R_0603_1608Metric, B.Cu at (342.0, 69.5)
- added UR0: Pro Micro, Keebio-Parts:ArduinoProMicro-ZigZag, B.Cu at (276.2, 166.7)
- added USBL1: USB C receptacle, Type-C:USB_C_GCT_USB4085, B.Cu at (36.7, 64.3)
- added USBR0: USB C receptacle, Type-C:USB_C_GCT_USB4085, B.Cu at (334.8, 64.3)
- moved JL0 0.48 mm to (55.3, 61.9)
- renumbered D00 to DL0, D01 to DL1, D10 to DL10, D11 to DL11, D12 to DL12, D13 to DL13, D14 to DL14, D15 to DL15, D16 to DL16, D02 to DL2, D20 to DL20, D21 to DL21, D22 to DL22, D23 to DL23, D24 to DL24, D25 to DL25, D26 to DL26, D03 to DL3, D30 to DL30, D31 to DL31, D32 to DL32, D33 to DL33, D34 to DL34, D35 to DL35, D36 to DL36, D04 to DL4, D43 to DL43, D44 to DL44, D45 to DL45, D46 to DL46, D05 to DL5, D54 to DL54, D55 to DL55, D56 to DL56, J0 to JL0, J1 to JL1, K00 to KL00, K01 to KL01, K02 to KL02, K03 to KL03, K04 to KL04, K05 to KL05, K10 to KL10, K11 to KL11, K12 to KL12, K13 to KL13, K14 to KL14, K15 to KL15, K16 to KL16, K20 to KL20, K21 to KL21, K22 to KL22, K23 to KL23, K24 to KL24, K25 to KL25, K26 to KL26, K30 to KL30, K31 to KL31, K32 to KL32, K33 to KL33, K34 to KL34, K35 to KL35, K36 to KL36, K43 to KL43, K44 to KL44, K45 to KL45, K46 to KL46, K54 to KL54, K55 to KL55, K56 to KL56, R0 to RL0, R1 to RL1, U0 to UL0
Routing:
- net Net-(JL0-Pad1): track 129.4 -> 122.4 mm
