File: splyd.kicad_pcb (KiCad board)
At the start: 2 copper layers, 156.2 x 146.6 mm, 148 parts

Commit message: Both halves fully wired
Parts:
- moved JR1 23.2 mm to (322.1, 143.5), turned to 100 degrees
- moved UR0 15.0 mm to (276.1, 151.6), turned to 190 degrees
- moved KR43 13.5 mm to (263.4, 134.5), turned to 10 degrees
- moved DR43 11.8 mm to (254.7, 139.9), turned to 100 degrees
- moved DR52 11.7 mm to (257.1, 158.8), turned to 100 degrees
- moved DR35 11.3 mm to (304.3, 136.7), turned to 90 degrees
- moved KR42 10.3 mm to (244.6, 137.8), turned to 10 degrees
- moved KR52 10.1 mm to (247.9, 156.6), turned to 10 degrees
- moved DL31 9.67 mm to (65.7, 137.1), turned to 90 degrees
- moved DR42 8.50 mm to (235.9, 143.2), turned to 100 degrees
- moved DR51 8.39 mm to (238.3, 162.1), turned to 100 degrees
- moved KR41 7.04 mm to (225.9, 141.1), turned to 10 degrees
- moved KR51 6.80 mm to (229.2, 159.9), turned to 10 degrees
- moved DR41 5.44 mm to (217.2, 146.5), turned to 100 degrees
- moved DR50 5.20 mm to (219.5, 165.5), turned to 100 degrees
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Routing:
- net Net-(DR10-Pad1): track 0.00 -> 271.3 mm, vias 0 -> 2
- net Net-(DR1-Pad1): track 0.00 -> 265.5 mm, vias 0 -> 2
- net Net-(DR20-Pad1): track 0.00 -> 255.9 mm, vias 0 -> 2
- net Net-(DR30-Pad1): track 0.00 -> 238.4 mm, vias 0 -> 2
- net Net-(KR10-Pad1): track 0.00 -> 163.0 mm, vias 0 -> 1
- net Net-(KR01-Pad1): track 0.00 -> 158.9 mm, vias 0 -> 1
- net Net-(KR06-Pad1): track 0.00 -> 152.3 mm, vias 0 -> 1
- net Net-(KR02-Pad1): track 0.00 -> 139.1 mm, vias 0 -> 1
- net Net-(KR05-Pad1): track 0.00 -> 134.2 mm, vias 0 -> 1
- net Net-(JR0-Pad2): track 0.00 -> 131.6 mm, vias 0 -> 1
- net Net-(KR04-Pad1): track 0.00 -> 129.4 mm, vias 0 -> 1
- net Net-(JR0-Pad3): track 0.00 -> 112.1 mm, vias 0 -> 1
- net Net-(JR0-Pad1): track 0.00 -> 109.8 mm, vias 0 -> 1
- net Net-(KR03-Pad1): track 0.00 -> 108.1 mm
- net Net-(JR1-Pad5): track 0.00 -> 105.7 mm, vias 0 -> 1
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Other:
- board size 156.2 x 146.6 mm -> 323.9 x 145.7 mm

Commit message: Keyswitch footprint with window and 3rd time routing
Parts:
- added REF**: MountingHole_3.2mm_M3, MountingHole:MountingHole_3.2mm_M3, F.Cu at (208.3, 71.0)
- added REF**: MountingHole_3.2mm_M3, MountingHole:MountingHole_3.2mm_M3, F.Cu at (27.3, 150.7)
- added REF**: MountingHole_3.2mm_M3, MountingHole:MountingHole_3.2mm_M3, F.Cu at (98.6, 163.6)
- added REF**: MountingHole_3.2mm_M3, MountingHole:MountingHole_3.2mm_M3, F.Cu at (169.9, 175.8)
- added REF**: MountingHole_3.2mm_M3, MountingHole:MountingHole_3.2mm_M3, F.Cu at (276.2, 37.1)
- added REF**: MountingHole_3.2mm_M3, MountingHole:MountingHole_3.2mm_M3, F.Cu at (344.3, 65.9)
- added REF**: MountingHole_3.2mm_M3, MountingHole:MountingHole_3.2mm_M3, F.Cu at (344.3, 150.7)
- added REF**: MountingHole_3.2mm_M3, MountingHole:MountingHole_3.2mm_M3, F.Cu at (272.9, 163.6)
- added REF**: MountingHole_3.2mm_M3, MountingHole:MountingHole_3.2mm_M3, F.Cu at (201.6, 175.8)
- added REF**: MountingHole_3.2mm_M3, MountingHole:MountingHole_3.2mm_M3, F.Cu at (27.3, 65.9)
- added REF**: MountingHole_3.2mm_M3, MountingHole:MountingHole_3.2mm_M3, F.Cu at (95.3, 37.1)
- added REF**: MountingHole_3.2mm_M3, MountingHole:MountingHole_3.2mm_M3, F.Cu at (163.3, 71.0)
- KL00, KL01, KL02, KL03, KL04, KL05, KL10, KL11, KL12, KL13, KL14, KL15, KL16, KL20, KL21, KL22, KL23, KL24, KL25, KL26, KL30, KL31, KL32, KL33, KL34, KL35, KL36, KL43, KL44, KL45, KL46, KL54, KL55, KL56, KR01, KR02, KR03, KR04, KR05, KR06, KR10, KR11, KR12, KR13, KR14, KR15, KR16, KR20, KR21, KR22, KR23, KR24, KR25, KR26, KR30, KR31, KR32, KR33, KR34, KR35, KR36, KR40, KR41, KR42, KR43, KR50, KR51, KR52: footprint keyswitches:Kailh_socket_MX -> keyswitches:Kailh_socket_MX--window
- moved RR1 14.1 mm to (327.9, 69.7)
- moved RL0 5.54 mm to (34.5, 72.0), turned to 0 degrees
- moved RR0 5.10 mm to (332.2, 72.0), turned to 0 degrees
- moved JL1 3.64 mm to (49.1, 142.3)
- moved UL0 2.67 mm to (97.9, 150.9)
- moved UR0 2.56 mm to (273.6, 150.9)
- moved JR1 1.28 mm to (322.4, 142.3)
- moved RL1 1.16 mm to (44.0, 68.4)
- moved JR0 1.14 mm to (317.4, 61.9)
- moved JL0 1.14 mm to (54.1, 61.9)
- moved DL56 0.14 mm to (151.1, 165.3)
Routing:
- net Net-(DL20-Pad1): track 263.6 -> 219.2 mm
- net Net-(DL10-Pad1): track 277.7 -> 233.9 mm
- net Net-(DL0-Pad1): track 271.1 -> 228.2 mm
- net Net-(DR1-Pad1): track 265.5 -> 240.0 mm
- net Net-(DR30-Pad1): track 238.4 -> 213.2 mm
- net Net-(DR20-Pad1): track 255.9 -> 233.3 mm
- net Net-(DR10-Pad1): track 271.3 -> 249.9 mm
- net Net-(DL30-Pad1): track 221.5 -> 203.1 mm, vias 1 -> 2
- net Net-(KR10-Pad1): track 163.0 -> 149.2 mm
- net Net-(KR02-Pad1): track 139.1 -> 125.5 mm
- net Net-(KR01-Pad1): track 158.9 -> 146.1 mm
- net Net-(KL03-Pad1): track 138.9 -> 126.8 mm, vias 1 -> 0
- net Net-(KL02-Pad1): track 131.3 -> 121.5 mm
- net Net-(KL04-Pad1): track 150.2 -> 140.7 mm
- net Net-(KR06-Pad1): track 152.3 -> 159.7 mm
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- removed copper zone on B.Cu, net Net-(JL1-Pad5)
- removed copper zone on F.Cu, net Net-(JL1-Pad5)
Other:
- board size 323.9 x 145.7 mm -> 325 x 145.9 mm

Commit message: Wire key RGB diodes for right thumb cluster
Parts:
- removed DL0, DL1, DL2, DL3, DL30, DL31, DL32, DL4, DL43, DL5, DL54, DL55, DL56, DR1, DR2, DR3, DR4, DR43, DR5, DR50, DR51, DR52, DR6: D, keyboard_parts:D_SOD123_axial
- removed KL30, KL31, KL32, KL43, KL54, KL55, KL56, KR43, KR50, KR51, KR52: KEYSW, keyswitches:Kailh_socket_MX--window
- removed the KR01 at (238.2, 60.9)
- removed the KR02 at (257.2, 56.2)
- removed the KR03 at (276.2, 48.6)
- removed the KR04 at (295.3, 57.1)
- removed the KR05 at (314.4, 76.2)
- removed the KR06 at (333.4, 80.0)
- removed the KR10 at (219.1, 81.9)
- removed the REF** at (208.3, 71.0)
- removed the REF** at (27.3, 150.7)
- removed the REF** at (98.6, 163.6)
- removed the REF** at (169.9, 175.8)
- removed the REF** at (276.2, 37.1)
- removed the REF** at (344.3, 65.9)
- removed the REF** at (344.3, 150.7)
- removed the REF** at (272.9, 163.6)
- removed the REF** at (201.6, 175.8)
- removed the REF** at (27.3, 65.9)
- removed the REF** at (95.3, 37.1)
- removed the REF** at (163.3, 71.0)
- added CL00: C_Small, Capacitor_SMD:C_0603_1608Metric_Pad1.05x0.95mm_HandSolder, F.Cu at (140.8, 36.4)
- added CL01: C_Small, Capacitor_SMD:C_0603_1608Metric_Pad1.05x0.95mm_HandSolder, F.Cu at (186.1, 23.0)
- added CL02: C_Small, Capacitor_SMD:C_0603_1608Metric_Pad1.05x0.95mm_HandSolder, B.Cu at (74.9, 83.2)
- added CL03: C_Small, Capacitor_SMD:C_0603_1608Metric_Pad1.05x0.95mm_HandSolder, F.Cu at (140.3, 46.1)
- added CL04: C_Small, Capacitor_SMD:C_0603_1608Metric_Pad1.05x0.95mm_HandSolder, F.Cu at (154.1, 42.3)
- added CL05: C_Small, Capacitor_SMD:C_0603_1608Metric_Pad1.05x0.95mm_HandSolder, F.Cu at (140.8, 33.9)
- added CL06: C_Small, Capacitor_SMD:C_0603_1608Metric_Pad1.05x0.95mm_HandSolder, F.Cu at (130.2, 39.1)
- added CL10: C_Small, Capacitor_SMD:C_0603_1608Metric_Pad1.05x0.95mm_HandSolder, F.Cu at (123.0, 19.5)
- added CL11: C_Small, Capacitor_SMD:C_0603_1608Metric_Pad1.05x0.95mm_HandSolder, F.Cu at (167.5, 13.1)
- added CL12: C_Small, Capacitor_SMD:C_0603_1608Metric_Pad1.05x0.95mm_HandSolder, F.Cu at (137.8, 27.2)
- added CL13: C_Small, Capacitor_SMD:C_0603_1608Metric_Pad1.05x0.95mm_HandSolder, F.Cu at (159.0, 17.2)
- added CL14: C_Small, Capacitor_SMD:C_0603_1608Metric_Pad1.05x0.95mm_HandSolder, F.Cu at (155.2, 7.22)
- added CL15: C_Small, Capacitor_SMD:C_0603_1608Metric_Pad1.05x0.95mm_HandSolder, F.Cu at (118.6, 19.5)
- added CL16: C_Small, Capacitor_SMD:C_0603_1608Metric_Pad1.05x0.95mm_HandSolder, F.Cu at (130.2, 36.6)
- added CL20: C_Small, Capacitor_SMD:C_0603_1608Metric_Pad1.05x0.95mm_HandSolder, F.Cu at (141.6, 18.6)
- added CL21: C_Small, Capacitor_SMD:C_0603_1608Metric_Pad1.05x0.95mm_HandSolder, F.Cu at (150.8, 9.73)
- added CL22: C_Small, Capacitor_SMD:C_0603_1608Metric_Pad1.05x0.95mm_HandSolder, F.Cu at (154.6, 19.7)
- added CL23: C_Small, Capacitor_SMD:C_0603_1608Metric_Pad1.05x0.95mm_HandSolder, F.Cu at (167.5, 10.6)
- added CL24: C_Small, Capacitor_SMD:C_0603_1608Metric_Pad1.05x0.95mm_HandSolder, F.Cu at (154.6, 17.2)
- added CL25: C_Small, Capacitor_SMD:C_0603_1608Metric_Pad1.05x0.95mm_HandSolder, F.Cu at (162.7, 24.7)
- added CL26: C_Small, Capacitor_SMD:C_0603_1608Metric_Pad1.05x0.95mm_HandSolder, F.Cu at (150.8, 7.22)
- added CL33: C_Small, Capacitor_SMD:C_0603_1608Metric_Pad1.05x0.95mm_HandSolder, F.Cu at (169.4, 22.8)
- added CL34: C_Small, Capacitor_SMD:C_0603_1608Metric_Pad1.05x0.95mm_HandSolder, F.Cu at (136.5, 35.4)
- added CL35: C_Small, Capacitor_SMD:C_0603_1608Metric_Pad1.05x0.95mm_HandSolder, F.Cu at (133.4, 27.2)
- added CL36: C_Small, Capacitor_SMD:C_0603_1608Metric_Pad1.05x0.95mm_HandSolder, F.Cu at (125.8, 39.1)
- added CL44: C_Small, Capacitor_SMD:C_0603_1608Metric_Pad1.05x0.95mm_HandSolder, F.Cu at (178.0, 10.3)
- added CL45: C_Small, Capacitor_SMD:C_0603_1608Metric_Pad1.05x0.95mm_HandSolder, F.Cu at (125.8, 36.6)
- added CL46: C_Small, Capacitor_SMD:C_0603_1608Metric_Pad1.05x0.95mm_HandSolder, F.Cu at (129.1, 27.2)
- added CLBC_32: C_Small, Capacitor_SMD:C_0603_1608Metric_Pad1.05x0.95mm_HandSolder, F.Cu at (132.8, 50.3)
- added CLBL_33: C_Small, Capacitor_SMD:C_0603_1608Metric_Pad1.05x0.95mm_HandSolder, F.Cu at (137.3, 18.6)
- added CLBR_29: C_Small, Capacitor_SMD:C_0603_1608Metric_Pad1.05x0.95mm_HandSolder, F.Cu at (164.8, 32.4)
- added CLTC_31: C_Small, Capacitor_SMD:C_0603_1608Metric_Pad1.05x0.95mm_HandSolder, F.Cu at (151.2, 31.0)
- added CLTL_34: C_Small, Capacitor_SMD:C_0603_1608Metric_Pad1.05x0.95mm_HandSolder, F.Cu at (120.6, 30.1)
- added CLTR_30: C_Small, Capacitor_SMD:C_0603_1608Metric_Pad1.05x0.95mm_HandSolder, F.Cu at (230.3, 43.0)
- added CR00: C_Small, Capacitor_SMD:C_0603_1608Metric_Pad1.05x0.95mm_HandSolder, F.Cu at (216.2, 28.7)
- added CR01: C_Small, Capacitor_SMD:C_0603_1608Metric_Pad1.05x0.95mm_HandSolder, F.Cu at (230.2, 14.3)
- added CR02: C_Small, Capacitor_SMD:C_0603_1608Metric_Pad1.05x0.95mm_HandSolder, F.Cu at (225.8, 18.5)
- added CR03: C_Small, Capacitor_SMD:C_0603_1608Metric_Pad1.05x0.95mm_HandSolder, F.Cu at (230.4, 9.85)
- added CR04: C_Small, Capacitor_SMD:C_0603_1608Metric_Pad1.05x0.95mm_HandSolder, F.Cu at (220.5, 23.9)
- added CR05: C_Small, Capacitor_SMD:C_0603_1608Metric_Pad1.05x0.95mm_HandSolder, F.Cu at (225.9, 14.3)
- added CR06: C_Small, Capacitor_SMD:C_0603_1608Metric_Pad1.05x0.95mm_HandSolder, F.Cu at (216.2, 23.9)
- added CR10: C_Small, Capacitor_SMD:C_0603_1608Metric_Pad1.05x0.95mm_HandSolder, F.Cu at (266.7, 10.0)
- added CR11: C_Small, Capacitor_SMD:C_0603_1608Metric_Pad1.05x0.95mm_HandSolder, F.Cu at (230.6, 5.24)
- added CR12: C_Small, Capacitor_SMD:C_0603_1608Metric_Pad1.05x0.95mm_HandSolder, F.Cu at (223.3, 49.1)
- added CR13: C_Small, Capacitor_SMD:C_0603_1608Metric_Pad1.05x0.95mm_HandSolder, F.Cu at (230.4, -0.13)
- added CR14: C_Small, Capacitor_SMD:C_0603_1608Metric_Pad1.05x0.95mm_HandSolder, F.Cu at (226.1, 9.85)
- added CR15: C_Small, Capacitor_SMD:C_0603_1608Metric_Pad1.05x0.95mm_HandSolder, F.Cu at (234.3, 49.9)
- added CR16: C_Small, Capacitor_SMD:C_0603_1608Metric_Pad1.05x0.95mm_HandSolder, F.Cu at (266.7, 5.03)
- added CR20: C_Small, Capacitor_SMD:C_0603_1608Metric_Pad1.05x0.95mm_HandSolder, F.Cu at (226.3, 5.24)
- added CR21: C_Small, Capacitor_SMD:C_0603_1608Metric_Pad1.05x0.95mm_HandSolder, F.Cu at (226.1, -0.13)
- added CR22: C_Small, Capacitor_SMD:C_0603_1608Metric_Pad1.05x0.95mm_HandSolder, F.Cu at (262.4, 10.0)
- added CR23: C_Small, Capacitor_SMD:C_0603_1608Metric_Pad1.05x0.95mm_HandSolder, F.Cu at (262.4, 5.03)
- added CR24: C_Small, Capacitor_SMD:C_0603_1608Metric_Pad1.05x0.95mm_HandSolder, F.Cu at (258.0, 10.0)
- added CR25: C_Small, Capacitor_SMD:C_0603_1608Metric_Pad1.05x0.95mm_HandSolder, F.Cu at (258.0, 5.03)
- added CR26: C_Small, Capacitor_SMD:C_0603_1608Metric_Pad1.05x0.95mm_HandSolder, F.Cu at (253.7, 10.0)
- added CR30: C_Small, Capacitor_SMD:C_0603_1608Metric_Pad1.05x0.95mm_HandSolder, B.Cu at (202.5, 150.1)
- added CR31: C_Small, Capacitor_SMD:C_0603_1608Metric_Pad1.05x0.95mm_HandSolder, B.Cu at (221.3, 146.8)
- added CR32: C_Small, Capacitor_SMD:C_0603_1608Metric_Pad1.05x0.95mm_HandSolder, B.Cu at (240.0, 143.5)
- added CR33: C_Small, Capacitor_SMD:C_0603_1608Metric_Pad1.05x0.95mm_HandSolder, B.Cu at (258.8, 140.2)
- added CR40: C_Small, Capacitor_SMD:C_0603_1608Metric_Pad1.05x0.95mm_HandSolder, B.Cu at (205.8, 168.8)
- added CR41: C_Small, Capacitor_SMD:C_0603_1608Metric_Pad1.05x0.95mm_HandSolder, B.Cu at (224.6, 165.5)
- added CR42: C_Small, Capacitor_SMD:C_0603_1608Metric_Pad1.05x0.95mm_HandSolder, B.Cu at (243.3, 162.2)
- added CRBC_30: C_Small, Capacitor_SMD:C_0603_1608Metric_Pad1.05x0.95mm_HandSolder, F.Cu at (255.5, 50.3)
- added CRBL_29: C_Small, Capacitor_SMD:C_0603_1608Metric_Pad1.05x0.95mm_HandSolder, F.Cu at (247.3, 50.3)
- added CRBR_33: C_Small, Capacitor_SMD:C_0603_1608Metric_Pad1.05x0.95mm_HandSolder, F.Cu at (265.0, 49.5)
- added CRTC_31: C_Small, Capacitor_SMD:C_0603_1608Metric_Pad1.05x0.95mm_HandSolder, F.Cu at (255.1, 38.6)
- added CRTL_30: C_Small, Capacitor_SMD:C_0603_1608Metric_Pad1.05x0.95mm_HandSolder, F.Cu at (245.6, 38.2)
- added CRTR_34: C_Small, Capacitor_SMD:C_0603_1608Metric_Pad1.05x0.95mm_HandSolder, F.Cu at (264.1, 38.3)
- added DL00: D, keyboard_parts:D_SOD123_axial, B.Cu at (29.9, 107.4)
- added DL00_1: SK6812MINI, keyboard_parts:SK6812MINIE-simple, F.Cu at (38.1, 107.6)
- added DL01: D, keyboard_parts:D_SOD123_axial, B.Cu at (49.2, 103.6)
- added DL01_6: SK6812MINI, keyboard_parts:SK6812MINIE-simple, F.Cu at (57.2, 103.8)
- added DL02: D, keyboard_parts:D_SOD123_axial, B.Cu at (68.2, 80.7)
- added DL02_7: SK6812MINI, keyboard_parts:SK6812MINIE-simple, F.Cu at (76.2, 80.9)
- added DL03: D, keyboard_parts:D_SOD123_axial, B.Cu at (86.9, 72.2)
- added DL03_12: SK6812MINI, keyboard_parts:SK6812MINIE-simple, F.Cu at (95.3, 72.4)
- added DL04: D, keyboard_parts:D_SOD123_axial, B.Cu at (105.9, 79.8)
- added DL04_13: SK6812MINI, keyboard_parts:SK6812MINIE-simple, F.Cu at (114.3, 80.0)
- added DL05: D, keyboard_parts:D_SOD123_axial, B.Cu at (125.0, 84.6)
- added DL05_18: SK6812MINI, keyboard_parts:SK6812MINIE-simple, F.Cu at (133.4, 84.7)
- added DL06: D, keyboard_parts:D_SOD123_axial, B.Cu at (144.0, 86.5)
- added DL06_19: SK6812MINI, keyboard_parts:SK6812MINIE-simple, F.Cu at (152.4, 86.7)
- added DL10_2: SK6812MINI, keyboard_parts:SK6812MINIE-simple, F.Cu at (38.1, 126.7)
- added DL11_5: SK6812MINI, keyboard_parts:SK6812MINIE-simple, F.Cu at (57.2, 122.8)
- added DL12_8: SK6812MINI, keyboard_parts:SK6812MINIE-simple, F.Cu at (76.2, 100.0)
- added DL13_11: SK6812MINI, keyboard_parts:SK6812MINIE-simple, F.Cu at (95.3, 91.4)
- added DL14_14: SK6812MINI, keyboard_parts:SK6812MINIE-simple, F.Cu at (114.3, 99.0)
- added DL15_17: SK6812MINI, keyboard_parts:SK6812MINIE-simple, F.Cu at (133.4, 103.8)
- added DL16_20: SK6812MINI, keyboard_parts:SK6812MINIE-simple, F.Cu at (152.4, 105.7)
- added DL20_3: SK6812MINI, keyboard_parts:SK6812MINIE-simple, F.Cu at (38.1, 145.7)
- added DL21_4: SK6812MINI, keyboard_parts:SK6812MINIE-simple, F.Cu at (57.2, 141.9)
- added DL22_9: SK6812MINI, keyboard_parts:SK6812MINIE-simple, F.Cu at (76.2, 119.0)
- added DL23_10: SK6812MINI, keyboard_parts:SK6812MINIE-simple, F.Cu at (95.3, 110.5)
- added DL24_15: SK6812MINI, keyboard_parts:SK6812MINIE-simple, F.Cu at (114.3, 118.1)
- added DL25_16: SK6812MINI, keyboard_parts:SK6812MINIE-simple, F.Cu at (133.4, 122.8)
- added DL26_21: SK6812MINI, keyboard_parts:SK6812MINIE-simple, F.Cu at (152.4, 124.8)
- added DL33_28: SK6812MINI, keyboard_parts:SK6812MINIE-simple, F.Cu at (106.9, 139.0)
- added DL34_27: SK6812MINI, keyboard_parts:SK6812MINIE-simple, F.Cu at (126.1, 142.5)
- added DL35_24: SK6812MINI, keyboard_parts:SK6812MINIE-simple, F.Cu at (144.4, 145.7)
- added DL36_23: SK6812MINI, keyboard_parts:SK6812MINIE-simple, F.Cu at (163.9, 148.8)
- added DL44_26: SK6812MINI, keyboard_parts:SK6812MINIE-simple, F.Cu at (123.3, 160.8)
- added DL45_25: SK6812MINI, keyboard_parts:SK6812MINIE-simple, F.Cu at (141.6, 164.0)
- added DL46_22: SK6812MINI, keyboard_parts:SK6812MINIE-simple, F.Cu at (160.4, 167.8)
- added DLBC_32: SK6812MINI, keyboard_parts:SK6812MINIE-simple_no-hole, F.Cu at (91.7, 138.3)
- added DLBL_33: SK6812MINI, keyboard_parts:SK6812MINIE-simple_no-hole, F.Cu at (38.1, 149.7)
- added DLBR_29: SK6812MINI, keyboard_parts:SK6812MINIE-simple_no-hole, F.Cu at (163.9, 152.8)
- added DLTC_31: SK6812MINI, keyboard_parts:SK6812MINIE-simple_no-hole, F.Cu at (95.3, 76.4)
- added DLTL_34: SK6812MINI, keyboard_parts:SK6812MINIE-simple_no-hole, F.Cu at (38.1, 111.6)
- added DLTR_30: SK6812MINI, keyboard_parts:SK6812MINIE-simple_no-hole, F.Cu at (152.4, 90.7)
- added DR00_19: SK6812MINI, keyboard_parts:SK6812MINIE-simple, F.Cu at (219.1, 86.7)
- added DR01_18: SK6812MINI, keyboard_parts:SK6812MINIE-simple, F.Cu at (238.2, 84.7)
- added DR02_13: SK6812MINI, keyboard_parts:SK6812MINIE-simple, F.Cu at (257.2, 80.0)
- added DR03_12: SK6812MINI, keyboard_parts:SK6812MINIE-simple, F.Cu at (276.2, 72.4)
- added DR04_7: SK6812MINI, keyboard_parts:SK6812MINIE-simple, F.Cu at (295.3, 80.9)
- added DR05_6: SK6812MINI, keyboard_parts:SK6812MINIE-simple, F.Cu at (314.4, 103.8)
- added DR06_1: SK6812MINI, keyboard_parts:SK6812MINIE-simple, F.Cu at (333.4, 107.6)
- added DR10_20: SK6812MINI, keyboard_parts:SK6812MINIE-simple, F.Cu at (219.1, 105.7)
- added DR11_17: SK6812MINI, keyboard_parts:SK6812MINIE-simple, F.Cu at (238.2, 103.8)
- added DR12_14: SK6812MINI, keyboard_parts:SK6812MINIE-simple, F.Cu at (257.2, 99.0)
- added DR13_11: SK6812MINI, keyboard_parts:SK6812MINIE-simple, F.Cu at (276.2, 91.4)
- added DR14_8: SK6812MINI, keyboard_parts:SK6812MINIE-simple, F.Cu at (295.3, 100.0)
- added DR15_5: SK6812MINI, keyboard_parts:SK6812MINIE-simple, F.Cu at (314.4, 122.8)
- added DR16_2: SK6812MINI, keyboard_parts:SK6812MINIE-simple, F.Cu at (333.4, 126.7)
- added DR20_21: SK6812MINI, keyboard_parts:SK6812MINIE-simple, F.Cu at (219.1, 124.8)
- added DR21_16: SK6812MINI, keyboard_parts:SK6812MINIE-simple, F.Cu at (238.0, 122.8)
- added DR22_15: SK6812MINI, keyboard_parts:SK6812MINIE-simple, F.Cu at (257.2, 118.1)
- added DR23_10: SK6812MINI, keyboard_parts:SK6812MINIE-simple, F.Cu at (276.2, 110.5)
- added DR24_9: SK6812MINI, keyboard_parts:SK6812MINIE-simple, F.Cu at (295.3, 119.0)
- added DR25_4: SK6812MINI, keyboard_parts:SK6812MINIE-simple, F.Cu at (314.4, 141.9)
- added DR26_3: SK6812MINI, keyboard_parts:SK6812MINIE-simple, F.Cu at (333.4, 145.7)
- added DR30: D, keyboard_parts:D_SOD123_axial, B.Cu at (199.8, 150.4)
- added DR30_23: SK6812MINI, keyboard_parts:SK6812MINIE-simple, F.Cu at (207.9, 149.1)
- added DR31: D, keyboard_parts:D_SOD123_axial, B.Cu at (217.2, 146.5)
- added DR31_24: SK6812MINI, keyboard_parts:SK6812MINIE-simple, F.Cu at (226.7, 145.8)
- added DR32: D, keyboard_parts:D_SOD123_axial, B.Cu at (235.9, 143.2)
- added DR32_27: SK6812MINI, keyboard_parts:SK6812MINIE-simple, F.Cu at (245.5, 142.5)
- added DR33: D, keyboard_parts:D_SOD123_axial, B.Cu at (254.7, 139.9)
- added DR33_28: SK6812MINI, keyboard_parts:SK6812MINIE-simple, F.Cu at (264.2, 139.2)
- added DR40_22: SK6812MINI, keyboard_parts:SK6812MINIE-simple, F.Cu at (211.3, 167.9)
- added DR41_25: SK6812MINI, keyboard_parts:SK6812MINIE-simple, F.Cu at (230.0, 164.6)
- added DR42_26: SK6812MINI, keyboard_parts:SK6812MINIE-simple, F.Cu at (248.8, 161.3)
- added DRBC_32: SK6812MINI, keyboard_parts:SK6812MINIE-simple_no-hole, F.Cu at (258.3, 50.5)
- added DRBL_29: SK6812MINI, keyboard_parts:SK6812MINIE-simple_no-hole, F.Cu at (250.0, 50.3)
- added DRBR_33: SK6812MINI, keyboard_parts:SK6812MINIE-simple_no-hole, F.Cu at (268.2, 49.5)
- added DRTC_31: SK6812MINI, keyboard_parts:SK6812MINIE-simple_no-hole, F.Cu at (257.8, 38.3)
- added DRTL_30: SK6812MINI, keyboard_parts:SK6812MINIE-simple_no-hole, F.Cu at (249.6, 38.3)
- added DRTR_34: SK6812MINI, keyboard_parts:SK6812MINIE-simple_no-hole, F.Cu at (267.5, 38.3)
- added KL06: KEYSW, keyswitches:Kailh_socket_MX--space, F.Cu at (152.4, 81.9)
- added KR00: KEYSW, keyswitches:Kailh_socket_MX--space, F.Cu at (219.1, 81.9)
- added KR30: KEYSW, keyswitches:Kailh_socket_MX--space, F.Cu at (207.1, 144.4)
- added KR31: KEYSW, keyswitches:Kailh_socket_MX--space, F.Cu at (225.9, 141.1)
- added KR32: KEYSW, keyswitches:Kailh_socket_MX--space, F.Cu at (244.6, 137.8)
- added KR33: KEYSW, keyswitches:Kailh_socket_MX--space, F.Cu at (263.4, 134.5)
- added REF**: MountingHole_3.2mm_M3_edge_distance, Mounting_Wuerth:MountingHole_3.2mm_M3_edge_distance, F.Cu at (28.6, 90.1)
- added REF**: MountingHole_3.2mm_M3_edge_distance, Mounting_Wuerth:MountingHole_3.2mm_M3_edge_distance, B.Cu at (339.5, 153.9)
- added REF**: MountingHole_3.2mm_M3_edge_distance, Mounting_Wuerth:MountingHole_3.2mm_M3_edge_distance, B.Cu at (273.1, 165.4)
- added REF**: MountingHole_3.2mm_M3_edge_distance, Mounting_Wuerth:MountingHole_3.2mm_M3_edge_distance, B.Cu at (206.6, 177.0)
- added REF**: MountingHole_3.2mm_M3_edge_distance, Mounting_Wuerth:MountingHole_3.2mm_M3_edge_distance, F.Cu at (158.5, 68.9)
- added REF**: MountingHole_3.2mm_M3_edge_distance, Mounting_Wuerth:MountingHole_3.2mm_M3_edge_distance, F.Cu at (95.3, 54.6)
- added REF**: MountingHole_3.2mm_M3_edge_distance, Mounting_Wuerth:MountingHole_3.2mm_M3_edge_distance, F.Cu at (32.0, 153.9)
- added REF**: MountingHole_3.2mm_M3_edge_distance, Mounting_Wuerth:MountingHole_3.2mm_M3_edge_distance, F.Cu at (98.5, 165.4)
- added REF**: MountingHole_3.2mm_M3_edge_distance, Mounting_Wuerth:MountingHole_3.2mm_M3_edge_distance, F.Cu at (164.9, 177.0)
- added REF**: MountingHole_3.2mm_M3_edge_distance, Mounting_Wuerth:MountingHole_3.2mm_M3_edge_distance, B.Cu at (213.0, 68.9)
- added REF**: MountingHole_3.2mm_M3_edge_distance, Mounting_Wuerth:MountingHole_3.2mm_M3_edge_distance, B.Cu at (276.2, 54.6)
- added REF**: MountingHole_3.2mm_M3_edge_distance, Mounting_Wuerth:MountingHole_3.2mm_M3_edge_distance, B.Cu at (342.9, 90.1)
- JL0, JR0: footprint mod_conn_av:jack_3.5_pj313d-smt -> Keebio-Parts:TRS-PJ-320B; moved to F.Cu
- KL00, KL01, KL02, KL03, KL04, KL05, KL10, KL11, KL12, KL13, KL14, KL15, KL16, KL20, KL21, KL22, KL23, KL24, KL25, KL26, KL33, KL34, KL35, KL36, KL44, KL45, KL46, KR40, KR41, KR42: footprint keyswitches:Kailh_socket_MX--window -> keyswitches:Kailh_socket_MX--space
- KR01: renamed from KR11; footprint keyswitches:Kailh_socket_MX--window -> keyswitches:Kailh_socket_MX--space
- KR02: renamed from KR12; footprint keyswitches:Kailh_socket_MX--window -> keyswitches:Kailh_socket_MX--space
- KR03: renamed from KR13; footprint keyswitches:Kailh_socket_MX--window -> keyswitches:Kailh_socket_MX--space
- KR04: renamed from KR14; footprint keyswitches:Kailh_socket_MX--window -> keyswitches:Kailh_socket_MX--space
- KR05: renamed from KR15; footprint keyswitches:Kailh_socket_MX--window -> keyswitches:Kailh_socket_MX--space
- KR06: renamed from KR16; footprint keyswitches:Kailh_socket_MX--window -> keyswitches:Kailh_socket_MX--space
- KR10: renamed from KR20; footprint keyswitches:Kailh_socket_MX--window -> keyswitches:Kailh_socket_MX--space
- KR11: renamed from KR21; footprint keyswitches:Kailh_socket_MX--window -> keyswitches:Kailh_socket_MX--space
- KR12: renamed from KR22; footprint keyswitches:Kailh_socket_MX--window -> keyswitches:Kailh_socket_MX--space
- KR13: renamed from KR23; footprint keyswitches:Kailh_socket_MX--window -> keyswitches:Kailh_socket_MX--space
- KR14: renamed from KR24; footprint keyswitches:Kailh_socket_MX--window -> keyswitches:Kailh_socket_MX--space
- KR15: renamed from KR25; footprint keyswitches:Kailh_socket_MX--window -> keyswitches:Kailh_socket_MX--space
- KR16: renamed from KR26; footprint keyswitches:Kailh_socket_MX--window -> keyswitches:Kailh_socket_MX--space
- KR20: renamed from KR30; footprint keyswitches:Kailh_socket_MX--window -> keyswitches:Kailh_socket_MX--space
- KR21: renamed from KR31; footprint keyswitches:Kailh_socket_MX--window -> keyswitches:Kailh_socket_MX--space
- KR22: renamed from KR32; footprint keyswitches:Kailh_socket_MX--window -> keyswitches:Kailh_socket_MX--space
- KR23: renamed from KR33; footprint keyswitches:Kailh_socket_MX--window -> keyswitches:Kailh_socket_MX--space
- KR24: renamed from KR34; footprint keyswitches:Kailh_socket_MX--window -> keyswitches:Kailh_socket_MX--space
- KR25: renamed from KR35; footprint keyswitches:Kailh_socket_MX--window -> keyswitches:Kailh_socket_MX--space
- KR26: renamed from KR36; footprint keyswitches:Kailh_socket_MX--window -> keyswitches:Kailh_socket_MX--space
- USBL1, USBR0: moved to F.Cu
- moved KL33 31.5 mm to (108.1, 134.5), turned to 350 degrees
- moved KL34 27.5 mm to (126.9, 137.8), turned to 350 degrees
- moved KL36 27.2 mm to (164.4, 144.4), turned to 350 degrees
- moved KL35 26.1 mm to (145.6, 141.1), turned to 350 degrees
- moved KL00 22.8 mm to (38.1, 102.8)
- moved KL01 22.8 mm to (57.2, 99.0)
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- renumbered DR10 to DR00, DR11 to DR01, DR12 to DR02, DR13 to DR03, DR14 to DR04, DR15 to DR05, DR16 to DR06, DR20 to DR10, DR21 to DR11, DR22 to DR12, DR23 to DR13, DR24 to DR14, DR25 to DR15, DR26 to DR16, DR30 to DR20, DR31 to DR21, DR32 to DR22, DR33 to DR23, DR34 to DR24, DR35 to DR25, DR36 to DR26
Connections:
- net Net-(JL0-Pad1) renamed GND1
- net Net-(JL0-Pad3) renamed L5V
- net Net-(JR0-Pad1) renamed GND2
- net Net-(JR0-Pad3) renamed R5V
- DL33 pad 1: Net-(DL30-Pad1) -> Net-(DL33-Pad1)
- DL34 pad 1: Net-(DL30-Pad1) -> Net-(DL33-Pad1)
- DL35 pad 1: Net-(DL30-Pad1) -> Net-(DL33-Pad1)
- DL36 pad 1: Net-(DL30-Pad1) -> Net-(DL33-Pad1)
- DL44 pad 1: Net-(DL43-Pad1) -> Net-(DL44-Pad1)
- DL45 pad 1: Net-(DL43-Pad1) -> Net-(DL44-Pad1)
- DL46 pad 1: Net-(DL43-Pad1) -> Net-(DL44-Pad1)
- UL0 pad 1: Net-(UL0-Pad1) -> LLED
- UL0 pad 10: Net-(DL30-Pad1) -> Net-(DL20-Pad1)
- UL0 pad 11: Net-(DL43-Pad1) -> Net-(DL33-Pad1)
- UL0 pad 12: Net-(DL54-Pad1) -> Net-(DL44-Pad1)
- UL0 pad 8: Net-(DL10-Pad1) -> Net-(DL00-Pad1)
- UL0 pad 9: Net-(DL20-Pad1) -> Net-(DL10-Pad1)
- UR0 pad 1: Net-(UR0-Pad1) -> RLED
- UR0 pad 11: Net-(DR40-Pad1) -> Net-(DR30-Pad1)
- UR0 pad 12: Net-(DR50-Pad1) -> Net-(DR40-Pad1)
Routing:
- net Net-(UR0-Pad7): track 240.0 -> 0.00 mm, vias 2 -> 0
- net Net-(DL00-Pad1): track 0.00 -> 228.7 mm, vias 0 -> 2
- net Net-(UL0-Pad7): track 228.2 -> 0.00 mm, vias 2 -> 0
- net Net-(DL30-Pad1): track 203.1 -> 0.00 mm, vias 2 -> 0
- net R5V: track 117.5 -> 292.3 mm, vias 1 -> 9
- net GND2: track 115.1 -> 266.8 mm, vias 1 -> 16
- net Net-(DR30-Pad1): track 0.00 -> 77.7 mm
- net Net-(DR20_21-Pad1): track 0.00 -> 60.1 mm
- net Net-(DL43-Pad1): track 59.5 -> 0.00 mm
- net Net-(DL33-Pad1): track 0.00 -> 59.5 mm
- net Net-(DL44-Pad1): track 0.00 -> 55.7 mm
- net Net-(DL54-Pad1): track 55.7 -> 0.00 mm
- net Net-(DR50-Pad1): track 42.5 -> 0.00 mm
- net Net-(JR0-Pad2): track 131.7 -> 102.9 mm
- net Net-(DR32_27-Pad3): track 0.00 -> 28.7 mm
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Other:
- board size 325 x 145.9 mm -> 324.2 x 132.5 mm

Commit message: Wire key RGB diodes for right thumb cluster with proper pinouts
Parts:
- DL00_1, DL01_6, DL02_7, DL03_12, DL04_13, DL05_18, DL06_19, DL10_2, DL11_5, DL12_8, DL13_11, DL14_14, DL15_17, DL16_20, DL20_3, DL21_4, DL22_9, DL23_10, DL24_15, DL25_16, DL26_21, DL33_28, DL34_27, DL35_24, DL36_23, DL44_26, DL45_25, DL46_22, DLBC_32, DLBL_33, DLBR_29, DLTC_31, DLTL_34, DLTR_30, DR00_19, DR01_18, DR02_13, DR03_12, DR04_7, DR05_6, DR06_1, DR10_20, DR11_17, DR12_14, DR13_11, DR14_8, DR15_5, DR16_2, DR20_21, DR21_16, DR22_15, DR23_10, DR24_9, DR25_4, DR26_3, DR30_23, DR31_24, DR32_27, DR33_28, DR40_22, DR41_25, DR42_26, DRBC_32, DRBL_29, DRBR_33, DRTC_31, DRTL_30, DRTR_34: value SK6812MINI -> SK6812MINI-E
- moved UR0 89.8 mm to (269.2, 240.6), turned to 180 degrees
- moved REF** 89.6 mm to (266.1, 254.8), turned to 170 degrees
- moved DR33_28 88.3 mm to (262.0, 227.4), turned to 270 degrees
- moved KR33 88.2 mm to (262.0, 222.7), turned to 0 degrees
- moved CR33 87.3 mm to (257.4, 227.4), turned to 270 degrees
- moved DR33 86.6 mm to (252.4, 226.5), turned to 90 degrees
- moved DR42_26 85.4 mm to (242.9, 246.5), turned to 270 degrees
- moved KR42 85.3 mm to (242.9, 241.7), turned to 0 degrees
- moved DR32_27 85.0 mm to (242.9, 227.4), turned to 270 degrees
- moved KR32 84.9 mm to (242.9, 222.7), turned to 0 degrees
- moved CR42 84.4 mm to (238.3, 246.5), turned to 270 degrees
- moved DR42 84.0 mm to (234.7, 246.3), turned to 90 degrees
- moved CR32 84.0 mm to (238.3, 227.4), turned to 270 degrees
- moved DR32 83.3 mm to (233.4, 226.5), turned to 90 degrees
- moved DR41_25 82.1 mm to (223.9, 246.5), turned to 270 degrees
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Connections:
- DL00_1 pad 1: Net-(DL00_1-Pad1) -> L5V
- DL00_1 pad 2: GND1 -> Net-(DL00_1-Pad2)
- DL00_1 pad 3: Net-(DL00_1-Pad3) -> GND1
- DL00_1 pad 4: L5V -> Net-(DL00_1-Pad4)
- DL01_6 pad 1: Net-(DL01_6-Pad1) -> L5V
- DL01_6 pad 2: GND1 -> Net-(DL01_6-Pad2)
- DL01_6 pad 3: Net-(DL01_6-Pad3) -> GND1
- DL01_6 pad 4: L5V -> Net-(DL01_6-Pad4)
- DL02_7 pad 1: Net-(DL02_7-Pad1) -> L5V
- DL02_7 pad 2: GND1 -> Net-(DL02_7-Pad2)
- DL02_7 pad 3: Net-(DL01_6-Pad1) -> GND1
- DL02_7 pad 4: L5V -> Net-(DL01_6-Pad2)
- DL03_12 pad 1: Net-(DL03_12-Pad1) -> L5V
- DL03_12 pad 2: GND1 -> Net-(DL03_12-Pad2)
- DL03_12 pad 3: Net-(DL03_12-Pad3) -> GND1
- DL03_12 pad 4: L5V -> Net-(DL03_12-Pad4)
- DL04_13 pad 1: Net-(DL04_13-Pad1) -> L5V
- DL04_13 pad 2: GND1 -> Net-(DL04_13-Pad2)
- DL04_13 pad 3: Net-(DL03_12-Pad1) -> GND1
- DL04_13 pad 4: L5V -> Net-(DL03_12-Pad2)
- DL05_18 pad 1: Net-(DL05_18-Pad1) -> L5V
- DL05_18 pad 2: GND1 -> Net-(DL05_18-Pad2)
- DL05_18 pad 3: Net-(DL05_18-Pad3) -> GND1
- DL05_18 pad 4: L5V -> Net-(DL05_18-Pad4)
- DL06_19 pad 1: Net-(DL06_19-Pad1) -> L5V
- DL06_19 pad 2: GND1 -> Net-(DL06_19-Pad2)
- DL06_19 pad 3: Net-(DL05_18-Pad1) -> GND1
- DL06_19 pad 4: L5V -> Net-(DL05_18-Pad2)
- DL10_2 pad 1: Net-(DL10_2-Pad1) -> L5V
- DL10_2 pad 2: GND1 -> Net-(DL10_2-Pad2)
- DL10_2 pad 3: Net-(DL00_1-Pad1) -> GND1
- DL10_2 pad 4: L5V -> Net-(DL00_1-Pad2)
- DL11_5 pad 1: Net-(DL01_6-Pad3) -> L5V
- DL11_5 pad 2: GND1 -> Net-(DL01_6-Pad4)
- DL11_5 pad 3: Net-(DL11_5-Pad3) -> GND1
- DL11_5 pad 4: L5V -> Net-(DL11_5-Pad4)
- DL12_8 pad 1: Net-(DL12_8-Pad1) -> L5V
- DL12_8 pad 2: GND1 -> Net-(DL12_8-Pad2)
- DL12_8 pad 3: Net-(DL02_7-Pad1) -> GND1
- DL12_8 pad 4: L5V -> Net-(DL02_7-Pad2)
- DL13_11 pad 1: Net-(DL03_12-Pad3) -> L5V
- DL13_11 pad 2: GND1 -> Net-(DL03_12-Pad4)
- DL13_11 pad 3: Net-(DL13_11-Pad3) -> GND1
- DL13_11 pad 4: L5V -> Net-(DL13_11-Pad4)
- DL14_14 pad 1: Net-(DL14_14-Pad1) -> L5V
- DL14_14 pad 2: GND1 -> Net-(DL14_14-Pad2)
- DL14_14 pad 3: Net-(DL04_13-Pad1) -> GND1
- DL14_14 pad 4: L5V -> Net-(DL04_13-Pad2)
- DL15_17 pad 1: Net-(DL05_18-Pad3) -> L5V
- DL15_17 pad 2: GND1 -> Net-(DL05_18-Pad4)
- DL15_17 pad 3: Net-(DL15_17-Pad3) -> GND1
- DL15_17 pad 4: L5V -> Net-(DL15_17-Pad4)
- DL16_20 pad 1: Net-(DL16_20-Pad1) -> L5V
- DL16_20 pad 2: GND1 -> Net-(DL16_20-Pad2)
- DL16_20 pad 3: Net-(DL06_19-Pad1) -> GND1
- DL16_20 pad 4: L5V -> Net-(DL06_19-Pad2)
- DL20_3 pad 1: Net-(DL20_3-Pad1) -> L5V
- DL20_3 pad 2: GND1 -> Net-(DL20_3-Pad2)
- DL20_3 pad 3: Net-(DL10_2-Pad1) -> GND1
- DL20_3 pad 4: L5V -> Net-(DL10_2-Pad2)
- DL21_4 pad 1: Net-(DL11_5-Pad3) -> L5V
- DL21_4 pad 2: GND1 -> Net-(DL11_5-Pad4)
- DL21_4 pad 3: Net-(DL20_3-Pad1) -> GND1
- DL21_4 pad 4: L5V -> Net-(DL20_3-Pad2)
- DL22_9 pad 1: Net-(DL22_9-Pad1) -> L5V
- DL22_9 pad 2: GND1 -> Net-(DL22_9-Pad2)
- DL22_9 pad 3: Net-(DL12_8-Pad1) -> GND1
- DL22_9 pad 4: L5V -> Net-(DL12_8-Pad2)
- DL23_10 pad 1: Net-(DL13_11-Pad3) -> L5V
- DL23_10 pad 2: GND1 -> Net-(DL13_11-Pad4)
- DL23_10 pad 3: Net-(DL22_9-Pad1) -> GND1
- DL23_10 pad 4: L5V -> Net-(DL22_9-Pad2)
- DL24_15 pad 1: Net-(DL24_15-Pad1) -> L5V
- DL24_15 pad 2: GND1 -> Net-(DL24_15-Pad2)
- DL24_15 pad 3: Net-(DL14_14-Pad1) -> GND1
- DL24_15 pad 4: L5V -> Net-(DL14_14-Pad2)
- DL25_16 pad 1: Net-(DL15_17-Pad3) -> L5V
- DL25_16 pad 2: GND1 -> Net-(DL15_17-Pad4)
- DL25_16 pad 3: Net-(DL24_15-Pad1) -> GND1
- DL25_16 pad 4: L5V -> Net-(DL24_15-Pad2)
- DL26_21 pad 1: Net-(DL26_21-Pad1) -> L5V
- DL26_21 pad 2: GND1 -> Net-(DL26_21-Pad2)
- DL26_21 pad 3: Net-(DL16_20-Pad1) -> GND1
- DL26_21 pad 4: L5V -> Net-(DL16_20-Pad2)
- DL33_28 pad 1: Net-(DL33_28-Pad1) -> L5V
- DL33_28 pad 2: GND1 -> Net-(DL33_28-Pad2)
- DL33_28 pad 3: Net-(DL33_28-Pad3) -> GND1
- DL33_28 pad 4: L5V -> Net-(DL33_28-Pad4)
- DL34_27 pad 1: Net-(DL33_28-Pad3) -> L5V
- DL34_27 pad 2: GND1 -> Net-(DL33_28-Pad4)
- DL34_27 pad 3: Net-(DL34_27-Pad3) -> GND1
- DL34_27 pad 4: L5V -> Net-(DL34_27-Pad4)
- DL35_24 pad 1: Net-(DL35_24-Pad1) -> L5V
- DL35_24 pad 2: GND1 -> Net-(DL35_24-Pad2)
- DL35_24 pad 3: Net-(DL35_24-Pad3) -> GND1
- DL35_24 pad 4: L5V -> Net-(DL35_24-Pad4)
- DL36_23 pad 1: Net-(DL35_24-Pad3) -> L5V
- DL36_23 pad 2: GND1 -> Net-(DL35_24-Pad4)
- DL36_23 pad 3: Net-(DL36_23-Pad3) -> GND1
- DL36_23 pad 4: L5V -> Net-(DL36_23-Pad4)
- DL44_26 pad 1: Net-(DL34_27-Pad3) -> L5V
- DL44_26 pad 2: GND1 -> Net-(DL34_27-Pad4)
- DL44_26 pad 3: Net-(DL44_26-Pad3) -> GND1
- DL44_26 pad 4: L5V -> Net-(DL44_26-Pad4)
- DL45_25 pad 1: Net-(DL44_26-Pad3) -> L5V
- DL45_25 pad 2: GND1 -> Net-(DL44_26-Pad4)
- DL45_25 pad 3: Net-(DL35_24-Pad1) -> GND1
- DL45_25 pad 4: L5V -> Net-(DL35_24-Pad2)
- DL46_22 pad 1: Net-(DL36_23-Pad3) -> L5V
- DL46_22 pad 2: GND1 -> Net-(DL36_23-Pad4)
- DL46_22 pad 3: Net-(DL26_21-Pad1) -> GND1
- DL46_22 pad 4: L5V -> Net-(DL26_21-Pad2)
- DLBC_32 pad 1: Net-(DLBC_32-Pad1) -> L5V
- DLBC_32 pad 2: GND1 -> Net-(DLBC_32-Pad2)
- DLBC_32 pad 3: Net-(DLBC_32-Pad3) -> GND1
- DLBC_32 pad 4: L5V -> Net-(DLBC_32-Pad4)
- DLBL_33 pad 1: Net-(DLBL_33-Pad1) -> L5V
- DLBL_33 pad 2: GND1 -> Net-(DLBL_33-Pad2)
- DLBL_33 pad 3: Net-(DLBC_32-Pad1) -> GND1
- DLBL_33 pad 4: L5V -> Net-(DLBC_32-Pad2)
- DLBR_29 pad 1: Net-(DLBR_29-Pad1) -> L5V
- DLBR_29 pad 2: GND1 -> Net-(DLBR_29-Pad2)
- DLBR_29 pad 3: LLED -> GND1
- DLBR_29 pad 4: L5V -> LLED
- DLTC_31 pad 1: Net-(DLBC_32-Pad3) -> L5V
- DLTC_31 pad 2: GND1 -> Net-(DLBC_32-Pad4)
- DLTC_31 pad 3: Net-(DLTC_31-Pad3) -> GND1
- DLTC_31 pad 4: L5V -> Net-(DLTC_31-Pad4)
- DLTL_34 pad 1: Net-(DL00_1-Pad3) -> L5V
- DLTL_34 pad 2: GND1 -> Net-(DL00_1-Pad4)
- DLTL_34 pad 3: Net-(DLBL_33-Pad1) -> GND1
- DLTL_34 pad 4: L5V -> Net-(DLBL_33-Pad2)
- DLTR_30 pad 1: Net-(DLTC_31-Pad3) -> L5V
- DLTR_30 pad 2: GND1 -> Net-(DLTC_31-Pad4)
- DLTR_30 pad 3: Net-(DLBR_29-Pad1) -> GND1
- DLTR_30 pad 4: L5V -> Net-(DLBR_29-Pad2)
- DR00_19 pad 1: Net-(DR00_19-Pad1) -> R5V
- DR00_19 pad 2: GND2 -> Net-(DR00_19-Pad2)
- DR00_19 pad 3: Net-(DR00_19-Pad3) -> GND2
- DR00_19 pad 4: R5V -> Net-(DR00_19-Pad4)
- DR01_18 pad 1: Net-(DR00_19-Pad3) -> R5V
- DR01_18 pad 2: GND2 -> Net-(DR00_19-Pad4)
- DR01_18 pad 3: Net-(DR01_18-Pad3) -> GND2
- DR01_18 pad 4: R5V -> Net-(DR01_18-Pad4)
- DR02_13 pad 1: Net-(DR02_13-Pad1) -> R5V
- DR02_13 pad 2: GND2 -> Net-(DR02_13-Pad2)
- DR02_13 pad 3: Net-(DR02_13-Pad3) -> GND2
- DR02_13 pad 4: R5V -> Net-(DR02_13-Pad4)
- DR03_12 pad 1: Net-(DR02_13-Pad3) -> R5V
- DR03_12 pad 2: GND2 -> Net-(DR02_13-Pad4)
- DR03_12 pad 3: Net-(DR03_12-Pad3) -> GND2
- DR03_12 pad 4: R5V -> Net-(DR03_12-Pad4)
- DR04_7 pad 1: Net-(DR04_7-Pad1) -> R5V
- DR04_7 pad 2: GND2 -> Net-(DR04_7-Pad2)
- DR04_7 pad 3: Net-(DR04_7-Pad3) -> GND2
- DR04_7 pad 4: R5V -> Net-(DR04_7-Pad4)
- DR05_6 pad 1: Net-(DR04_7-Pad3) -> R5V
- DR05_6 pad 2: GND2 -> Net-(DR04_7-Pad4)
- DR05_6 pad 3: Net-(DR05_6-Pad3) -> GND2
- DR05_6 pad 4: R5V -> Net-(DR05_6-Pad4)
- DR06_1 pad 1: Net-(DR06_1-Pad1) -> R5V
- DR06_1 pad 2: GND2 -> Net-(DR06_1-Pad2)
- DR06_1 pad 3: Net-(DR06_1-Pad3) -> GND2
- DR06_1 pad 4: R5V -> Net-(DR06_1-Pad4)
- DR10_20 pad 1: Net-(DR10_20-Pad1) -> R5V
- DR10_20 pad 2: GND2 -> Net-(DR10_20-Pad2)
- DR10_20 pad 3: Net-(DR00_19-Pad1) -> GND2
- DR10_20 pad 4: R5V -> Net-(DR00_19-Pad2)
- DR11_17 pad 1: Net-(DR01_18-Pad3) -> R5V
- DR11_17 pad 2: GND2 -> Net-(DR01_18-Pad4)
- DR11_17 pad 3: Net-(DR11_17-Pad3) -> GND2
- DR11_17 pad 4: R5V -> Net-(DR11_17-Pad4)
- DR12_14 pad 1: Net-(DR12_14-Pad1) -> R5V
- DR12_14 pad 2: GND2 -> Net-(DR12_14-Pad2)
- DR12_14 pad 3: Net-(DR02_13-Pad1) -> GND2
- DR12_14 pad 4: R5V -> Net-(DR02_13-Pad2)
- DR13_11 pad 1: Net-(DR03_12-Pad3) -> R5V
- DR13_11 pad 2: GND2 -> Net-(DR03_12-Pad4)
- DR13_11 pad 3: Net-(DR13_11-Pad3) -> GND2
- DR13_11 pad 4: R5V -> Net-(DR13_11-Pad4)
- DR14_8 pad 1: Net-(DR14_8-Pad1) -> R5V
- DR14_8 pad 2: GND2 -> Net-(DR14_8-Pad2)
- DR14_8 pad 3: Net-(DR04_7-Pad1) -> GND2
- DR14_8 pad 4: R5V -> Net-(DR04_7-Pad2)
- DR15_5 pad 1: Net-(DR05_6-Pad3) -> R5V
- DR15_5 pad 2: GND2 -> Net-(DR05_6-Pad4)
- DR15_5 pad 3: Net-(DR15_5-Pad3) -> GND2
- DR15_5 pad 4: R5V -> Net-(DR15_5-Pad4)
- DR16_2 pad 1: Net-(DR16_2-Pad1) -> R5V
- DR16_2 pad 2: GND2 -> Net-(DR16_2-Pad2)
- DR16_2 pad 3: Net-(DR06_1-Pad1) -> GND2
- DR16_2 pad 4: R5V -> Net-(DR06_1-Pad2)
- DR20_21 pad 1: Net-(DR20_21-Pad1) -> R5V
- DR20_21 pad 2: GND2 -> Net-(DR20_21-Pad2)
- DR20_21 pad 3: Net-(DR10_20-Pad1) -> GND2
- DR20_21 pad 4: R5V -> Net-(DR10_20-Pad2)
- DR21_16 pad 1: Net-(DR11_17-Pad3) -> R5V
- DR21_16 pad 2: GND2 -> Net-(DR11_17-Pad4)
- DR21_16 pad 3: Net-(DR21_16-Pad3) -> GND2
- DR21_16 pad 4: R5V -> Net-(DR21_16-Pad4)
- DR22_15 pad 1: Net-(DR21_16-Pad3) -> R5V
- DR22_15 pad 2: GND2 -> Net-(DR21_16-Pad4)
- DR22_15 pad 3: Net-(DR12_14-Pad1) -> GND2
- DR22_15 pad 4: R5V -> Net-(DR12_14-Pad2)
- DR23_10 pad 1: Net-(DR13_11-Pad3) -> R5V
- DR23_10 pad 2: GND2 -> Net-(DR13_11-Pad4)
- DR23_10 pad 3: Net-(DR23_10-Pad3) -> GND2
- DR23_10 pad 4: R5V -> Net-(DR23_10-Pad4)
- DR24_9 pad 1: Net-(DR23_10-Pad3) -> R5V
- DR24_9 pad 2: GND2 -> Net-(DR23_10-Pad4)
- DR24_9 pad 3: Net-(DR14_8-Pad1) -> GND2
- DR24_9 pad 4: R5V -> Net-(DR14_8-Pad2)
- DR25_4 pad 1: Net-(DR15_5-Pad3) -> R5V
- DR25_4 pad 2: GND2 -> Net-(DR15_5-Pad4)
- DR25_4 pad 3: Net-(DR25_4-Pad3) -> GND2
- DR25_4 pad 4: R5V -> Net-(DR25_4-Pad4)
- DR26_3 pad 1: Net-(DR25_4-Pad3) -> R5V
- DR26_3 pad 2: GND2 -> Net-(DR25_4-Pad4)
- DR26_3 pad 3: Net-(DR16_2-Pad1) -> GND2
- DR26_3 pad 4: R5V -> Net-(DR16_2-Pad2)
- DR30_23 pad 1: Net-(DR30_23-Pad1) -> R5V
- DR30_23 pad 2: GND2 -> Net-(DR30_23-Pad2)
- DR30_23 pad 3: Net-(DR30_23-Pad3) -> GND2
- DR30_23 pad 4: R5V -> Net-(DR30_23-Pad4)
- DR31_24 pad 1: Net-(DR31_24-Pad1) -> R5V
- DR31_24 pad 2: GND2 -> Net-(DR31_24-Pad2)
- DR31_24 pad 3: Net-(DR30_23-Pad1) -> GND2
- DR31_24 pad 4: R5V -> Net-(DR30_23-Pad2)
- DR32_27 pad 1: Net-(DR32_27-Pad1) -> R5V
- DR32_27 pad 2: GND2 -> Net-(DR32_27-Pad2)
- DR32_27 pad 3: Net-(DR32_27-Pad3) -> GND2
- DR32_27 pad 4: R5V -> Net-(DR32_27-Pad4)
- DR33_28 pad 1: Net-(DR33_28-Pad1) -> R5V
- DR33_28 pad 2: GND2 -> Net-(DR33_28-Pad2)
- DR33_28 pad 3: Net-(DR32_27-Pad1) -> GND2
- DR33_28 pad 4: R5V -> Net-(DR32_27-Pad2)
- DR40_22 pad 1: Net-(DR30_23-Pad3) -> R5V
- DR40_22 pad 2: GND2 -> Net-(DR30_23-Pad4)
- DR40_22 pad 3: Net-(DR20_21-Pad1) -> GND2
- DR40_22 pad 4: R5V -> Net-(DR20_21-Pad2)
- DR41_25 pad 1: Net-(DR41_25-Pad1) -> R5V
- DR41_25 pad 2: GND2 -> Net-(DR41_25-Pad2)
- DR41_25 pad 3: Net-(DR31_24-Pad1) -> GND2
- DR41_25 pad 4: R5V -> Net-(DR31_24-Pad2)
- DR42_26 pad 1: Net-(DR32_27-Pad3) -> R5V
- DR42_26 pad 2: GND2 -> Net-(DR32_27-Pad4)
- DR42_26 pad 3: Net-(DR41_25-Pad1) -> GND2
- DR42_26 pad 4: R5V -> Net-(DR41_25-Pad2)
- DRBC_32 pad 1: Net-(DRBC_32-Pad1) -> R5V
- DRBC_32 pad 2: GND2 -> Net-(DRBC_32-Pad2)
- DRBC_32 pad 3: Net-(DRBC_32-Pad3) -> GND2
- DRBC_32 pad 4: R5V -> Net-(DRBC_32-Pad4)
- DRBL_29 pad 1: Net-(DRBL_29-Pad1) -> R5V
- DRBL_29 pad 2: GND2 -> Net-(DRBL_29-Pad2)
- DRBL_29 pad 3: RLED -> GND2
- DRBL_29 pad 4: R5V -> RLED
- DRBR_33 pad 1: Net-(DRBR_33-Pad1) -> R5V
- DRBR_33 pad 2: GND2 -> Net-(DRBR_33-Pad2)
- DRBR_33 pad 3: Net-(DRBC_32-Pad1) -> GND2
- DRBR_33 pad 4: R5V -> Net-(DRBC_32-Pad2)
- DRTC_31 pad 1: Net-(DRBC_32-Pad3) -> R5V
- DRTC_31 pad 2: GND2 -> Net-(DRBC_32-Pad4)
- DRTC_31 pad 3: Net-(DRTC_31-Pad3) -> GND2
- DRTC_31 pad 4: R5V -> Net-(DRTC_31-Pad4)
- DRTL_30 pad 1: Net-(DRTC_31-Pad3) -> R5V
- DRTL_30 pad 2: GND2 -> Net-(DRTC_31-Pad4)
- DRTL_30 pad 3: Net-(DRBL_29-Pad1) -> GND2
- DRTL_30 pad 4: R5V -> Net-(DRBL_29-Pad2)
- DRTR_34 pad 1: Net-(DR06_1-Pad3) -> R5V
- DRTR_34 pad 2: GND2 -> Net-(DR06_1-Pad4)
- DRTR_34 pad 3: Net-(DRBR_33-Pad1) -> GND2
- DRTR_34 pad 4: R5V -> Net-(DRBR_33-Pad2)
Routing:
- net Net-(DR20_21-Pad1): track 60.1 -> 0.00 mm
- net Net-(DR30_23-Pad4): track 0.00 -> 32.8 mm
- net Net-(DR32_27-Pad4): track 0.00 -> 32.7 mm
- net Net-(DR41_25-Pad2): track 0.00 -> 32.5 mm
- net Net-(DR32_27-Pad2): track 0.00 -> 30.1 mm, vias 0 -> 2
- net Net-(DR30_23-Pad2): track 0.00 -> 30.0 mm, vias 0 -> 2
- net Net-(DR32_27-Pad3): track 28.7 -> 0.00 mm
- net Net-(DR30_23-Pad3): track 28.7 -> 0.00 mm
- net Net-(DR31_24-Pad2): track 0.00 -> 21.1 mm
- net Net-(DR31_24-Pad1): track 19.7 -> 0.00 mm
- net Net-(DR30_23-Pad1): track 14.5 -> 0.00 mm, vias 2 -> 0
- net Net-(DR41_25-Pad1): track 14.5 -> 0.00 mm
- net Net-(DR32_27-Pad1): track 14.5 -> 0.00 mm, vias 2 -> 0
- net R5V: track 292.3 -> 283.9 mm
- net GND2: track 266.8 -> 272.4 mm
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Other:
- board size 324.2 x 132.5 mm -> 324.2 x 209.9 mm
