File: splyd.kicad_pcb (KiCad board)
At the start: 2 copper layers, 324.2 x 132.5 mm, 274 parts

Commit message: Wire LED data to more suitable pin (shifts all row pins by 1)
Parts:
- CL00, CL01, CL03, CL04, CL05, CL06, CL10, CL11, CL12, CL13, CL14, CL15, CL16, CL20, CL21, CL22, CL23, CL24, CL25, CL26, CLBL_33, CLTC_31, CLTL_34, CLTR_30, CR00, CR01, CR02, CR03, CR04, CR05, CR06, CR10, CR11, CR12, CR13, CR14, CR16, CR20, CR21, CR22, CR23, CR24, CR25, CR26, CRTC_31, CRTL_30, CRTR_34: moved to B.Cu
- moved CRTL_30 10.3 mm to (214.5, 91.4), turned to 90 degrees
- moved CLBL_33 6.20 mm to (37.7, 149.7), turned to 90 degrees
- moved CRTR_34 4.59 mm to (328.8, 112.2), turned to 90 degrees
- moved CRTC_31 4.20 mm to (271.9, 77.1), turned to 90 degrees
- moved CR25 3.24 mm to (309.8, 141.9), turned to 270 degrees
- moved CL04 3.24 mm to (109.8, 80.0), turned to 270 degrees
- moved CR03 3.07 mm to (271.7, 72.4), turned to 270 degrees
- moved CR21 3.07 mm to (233.4, 122.8), turned to 270 degrees
- moved CL25 3.05 mm to (128.8, 122.8), turned to 270 degrees
- moved CR10 3.05 mm to (214.5, 105.7), turned to 270 degrees
- moved CL26 3.05 mm to (147.9, 124.8), turned to 270 degrees
- moved CR13 3.05 mm to (271.7, 91.4), turned to 270 degrees
- moved CL01 3.01 mm to (52.6, 103.8), turned to 270 degrees
- moved CL03 2.96 mm to (90.7, 72.4), turned to 270 degrees
- moved CR06 2.96 mm to (328.8, 107.6), turned to 270 degrees
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Connections:
- R_LLED1 pad 1: LLED -> Net-(R_LLED1-Pad1)
- R_LLED1 pad 2: Net-(R_LLED1-Pad2) -> LLED
- UL0 pad 1: Net-(R_LLED1-Pad2) -> Net-(UL0-Pad1)
- UL0 pad 10: Net-(DL20-Pad1) -> Net-(DL33-Pad1)
- UL0 pad 11: Net-(DL33-Pad1) -> Net-(DL44-Pad1)
- UL0 pad 12: Net-(DL44-Pad1) -> Net-(R_LLED1-Pad1)
- UL0 pad 7: Net-(UL0-Pad7) -> Net-(DL00-Pad1)
- UL0 pad 8: Net-(DL00-Pad1) -> Net-(DL10-Pad1)
- UL0 pad 9: Net-(DL10-Pad1) -> Net-(DL20-Pad1)
- UR0 pad 1: Net-(R_RLED1-Pad1) -> Net-(UR0-Pad1)
- UR0 pad 10: Net-(DR20-Pad1) -> Net-(DR30-Pad1)
- UR0 pad 11: Net-(DR30-Pad1) -> Net-(DR40-Pad1)
- UR0 pad 12: Net-(DR40-Pad1) -> Net-(R_RLED1-Pad1)
- UR0 pad 7: Net-(UR0-Pad7) -> Net-(DR00-Pad1)
- UR0 pad 8: Net-(DR00-Pad1) -> Net-(DR10-Pad1)
- UR0 pad 9: Net-(DR10-Pad1) -> Net-(DR20-Pad1)
Routing:
- net GND2: track 312.7 -> 563.2 mm, vias 19 -> 37
- net R5V: track 313.8 -> 559.3 mm, vias 12 -> 23
- net Net-(R_LLED1-Pad2): track 74.5 -> 0.00 mm, vias 2 -> 0
- net Net-(DRBR_33-Pad2): track 0.00 -> 45.2 mm
- net Net-(R_LLED1-Pad1): track 0.00 -> 41.3 mm, vias 0 -> 1
- net Net-(KR06-Pad1): track 103.3 -> 136.2 mm, vias 0 -> 1
- net Net-(R_RLED1-Pad1): track 82.9 -> 51.2 mm, vias 3 -> 2
- net Net-(DR16_2-Pad2): track 0.00 -> 19.7 mm
- net Net-(DR25_4-Pad4): track 0.00 -> 16.2 mm, vias 0 -> 2
- net Net-(DR20-Pad1): track 203.1 -> 199.0 mm
- net Net-(DR10-Pad1): track 219.6 -> 216.9 mm
- net Net-(DL10-Pad1): track 213.6 -> 210.8 mm
- net Net-(DL20-Pad1): track 201.2 -> 198.9 mm
- net Net-(DR40-Pad1): track 59.5 -> 61.9 mm
- net Net-(DL00-Pad1): track 228.7 -> 226.3 mm
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
Commit message: Wire all LEDs on right half
Parts:
- moved CRTC_31 0.19 mm to (271.7, 77.1)
- moved DRTC_31 0.19 mm to (276.2, 77.1)
Routing:
- net R5V: track 559.3 -> 821.1 mm, vias 23 -> 42
- net GND2: track 563.2 -> 794.4 mm, vias 37 -> 67
- net Net-(DRBC_32-Pad4): track 0.00 -> 71.6 mm, vias 0 -> 2
- net Net-(DRBC_32-Pad2): track 0.00 -> 68.4 mm, vias 0 -> 2
- net Net-(DRTC_31-Pad4): track 0.00 -> 68.3 mm, vias 0 -> 2
- net Net-(DRBL_29-Pad2): track 38.8 -> 85.4 mm, vias 0 -> 2
- net Net-(DR04_7-Pad4): track 0.00 -> 33.6 mm, vias 0 -> 2
- net Net-(DR03_12-Pad4): track 0.00 -> 27.8 mm
- net Net-(DR11_17-Pad4): track 0.00 -> 27.5 mm
- net Net-(DR05_6-Pad4): track 0.00 -> 27.4 mm
- net Net-(DR01_18-Pad4): track 0.00 -> 27.4 mm
- net Net-(DR15_5-Pad4): track 0.00 -> 27.4 mm
- net Net-(DR13_11-Pad4): track 0.00 -> 27.4 mm
- net Net-(DR12_14-Pad2): track 0.00 -> 19.7 mm
- net Net-(DR02_13-Pad2): track 0.00 -> 19.7 mm
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
Commit message: Complete trace routing
Parts:
- moved DL21 0.82 mm to (65.6, 141.7)
Routing:
- net L5V: track 306.3 -> 816.0 mm, vias 12 -> 42
- net GND1: track 314.7 -> 797.0 mm, vias 18 -> 65
- net Net-(DLBC_32-Pad4): track 0.00 -> 69.9 mm
- net Net-(DLTC_31-Pad4): track 0.00 -> 62.2 mm, vias 0 -> 2
- net Net-(DLBC_32-Pad2): track 0.00 -> 59.3 mm
- net Net-(DL01_6-Pad2): track 0.00 -> 46.8 mm, vias 0 -> 2
- net Net-(DLBL_33-Pad2): track 0.00 -> 38.9 mm
- net Net-(DLBR_29-Pad2): track 28.5 -> 67.3 mm, vias 0 -> 2
- net Net-(DL03_12-Pad2): track 0.00 -> 37.0 mm, vias 0 -> 2
- net Net-(DL22_9-Pad2): track 0.00 -> 35.8 mm, vias 0 -> 2
- net Net-(DL24_15-Pad2): track 0.00 -> 34.5 mm, vias 0 -> 2
- net Net-(DL20_3-Pad2): track 0.00 -> 33.7 mm
- net Net-(DL05_18-Pad2): track 0.00 -> 33.1 mm, vias 0 -> 2
- net Net-(DL03_12-Pad4): track 0.00 -> 27.9 mm
- net Net-(DL15_17-Pad4): track 0.00 -> 27.4 mm
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
Commit message: Fill ground planes and panelize
Parts:
- removed the REF** at (339.5, 153.9)
- removed the REF** at (273.1, 165.4)
- removed the REF** at (206.6, 177.0)
- removed the REF** at (213.0, 68.9)
- removed the REF** at (276.2, 54.6)
- removed the REF** at (342.9, 90.1)
- added REF**: breakaway-mousebites-tangent, Keebio-Parts:breakaway-mousebites-tangent, F.Cu at (182.5, 185.3)
- added REF**: breakaway-mousebites-tangent, Keebio-Parts:breakaway-mousebites-tangent, F.Cu at (37.0, 78.8)
- added REF**: breakaway-mousebites-tangent, Keebio-Parts:breakaway-mousebites-tangent, F.Cu at (95.3, 49.9)
- added REF**: MountingHole_3.2mm_M3_edge_distance, Mounting_Wuerth:MountingHole_3.2mm_M3_edge_distance, B.Cu at (205.4, 68.9)
- added REF**: MountingHole_3.2mm_M3_edge_distance, Mounting_Wuerth:MountingHole_3.2mm_M3_edge_distance, B.Cu at (268.6, 54.6)
- added REF**: breakaway-mousebites-tangent, Keebio-Parts:breakaway-mousebites-tangent, F.Cu at (268.6, 49.9)
- added REF**: MountingHole_3.2mm_M3_edge_distance, Mounting_Wuerth:MountingHole_3.2mm_M3_edge_distance, B.Cu at (335.3, 90.1)
- added REF**: MountingHole_3.2mm_M3_edge_distance, Mounting_Wuerth:MountingHole_3.2mm_M3_edge_distance, B.Cu at (331.9, 153.9)
- added REF**: MountingHole_3.2mm_M3_edge_distance, Mounting_Wuerth:MountingHole_3.2mm_M3_edge_distance, B.Cu at (265.4, 165.4)
- added REF**: MountingHole_3.2mm_M3_edge_distance, Mounting_Wuerth:MountingHole_3.2mm_M3_edge_distance, B.Cu at (199.0, 177.0)
- added REF**: breakaway-mousebites-tangent, Keebio-Parts:breakaway-mousebites-tangent, F.Cu at (337.0, 49.9)
- added REF**: breakaway-mousebites-tangent, Keebio-Parts:breakaway-mousebites-tangent, F.Cu at (326.9, 78.8)
- added REF**: breakaway-mousebites-tangent, Keebio-Parts:breakaway-mousebites-tangent, B.Cu at (319.5, 160.9)
- added REF**: breakaway-mousebites-tangent, Keebio-Parts:breakaway-mousebites-tangent, B.Cu at (220.7, 178.1)
- added REF**: breakaway-mousebites-tangent, Keebio-Parts:breakaway-mousebites-tangent, F.Cu at (26.9, 49.9)
- added REF**: breakaway-mousebites-tangent, Keebio-Parts:breakaway-mousebites-tangent, F.Cu at (44.4, 160.9)
- added REF**: breakaway-mousebites-tangent, Keebio-Parts:breakaway-mousebites-tangent, F.Cu at (143.2, 178.1)
- moved CR33 7.62 mm to (252.1, 140.0)
- moved KR33 7.62 mm to (255.8, 134.5)
- moved CR00 7.62 mm to (206.9, 86.7)
- moved CR01 7.62 mm to (226.0, 84.7)
- moved CR03 7.62 mm to (264.1, 72.4)
- moved CR04 7.62 mm to (283.1, 80.9)
- moved CR05 7.62 mm to (302.2, 103.8)
- moved CR10 7.62 mm to (206.9, 105.7)
- moved CR11 7.62 mm to (226.0, 103.8)
- moved CR13 7.62 mm to (264.1, 91.4)
- moved CR14 7.62 mm to (283.1, 100.0)
- moved CR15 7.62 mm to (302.2, 122.8)
- moved CR20 7.62 mm to (206.9, 124.8)
- moved CR23 7.62 mm to (264.1, 110.5)
- moved CR24 7.62 mm to (283.1, 119.0)
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Connections:
- JL1 pad 5: Net-(JL1-Pad5) -> GND1
- JR1 pad 5: Net-(JR1-Pad5) -> GND2
- RL0 pad 1: Net-(JL1-Pad5) -> GND1
- RL1 pad 1: Net-(JL1-Pad5) -> GND1
- RR0 pad 1: Net-(JR1-Pad5) -> GND2
- RR1 pad 1: Net-(JR1-Pad5) -> GND2
- USBL1 pad A1: Net-(JL1-Pad5) -> GND1
- USBL1 pad A12: Net-(JL1-Pad5) -> GND1
- USBL1 pad B1: Net-(JL1-Pad5) -> GND1
- USBL1 pad B12: Net-(JL1-Pad5) -> GND1
- USBL1 pad S1: Net-(JL1-Pad5) -> GND1
- USBR0 pad A1: Net-(JR1-Pad5) -> GND2
- USBR0 pad A12: Net-(JR1-Pad5) -> GND2
- USBR0 pad B1: Net-(JR1-Pad5) -> GND2
- USBR0 pad B12: Net-(JR1-Pad5) -> GND2
- USBR0 pad S1: Net-(JR1-Pad5) -> GND2
Routing:
- net GND1: track 797.0 -> 886.5 mm, vias 65 -> 68
- net Net-(JL1-Pad5): track 89.5 -> 0.00 mm
- net GND2: track 795.0 -> 879.8 mm, vias 67 -> 66
- net Net-(JR1-Pad5): track 83.8 -> 0.00 mm
- added copper zone on B.Cu, net GND1
- added copper zone on F.Cu, net GND1
- added copper zone on B.Cu, net GND2
- added copper zone on F.Cu, net GND2
Other:
- board size 324.2 x 132.5 mm -> 316.6 x 144.6 mm
- board text added: "JLCJLCJLCJLC"

Commit message: Edge cut rework and prep for case design
Parts:
- removed the REF** at (182.5, 185.3)
- removed the REF** at (28.6, 90.1)
- removed the REF** at (158.5, 68.9)
- removed the REF** at (95.3, 54.6)
- removed the REF** at (32.0, 153.9)
- removed the REF** at (98.5, 165.4)
- removed the REF** at (164.9, 177.0)
- removed the REF** at (205.4, 68.9)
- removed the REF** at (268.6, 54.6)
- removed the REF** at (268.6, 49.9)
- removed the REF** at (335.3, 90.1)
- removed the REF** at (331.9, 153.9)
- removed the REF** at (265.4, 165.4)
- removed the REF** at (199.0, 177.0)
- removed the REF** at (337.0, 49.9)
- removed the REF** at (326.9, 78.8)
- removed the REF** at (319.5, 160.9)
- removed the REF** at (220.7, 178.1)
- removed the REF** at (44.4, 160.9)
- removed the REF** at (143.2, 178.1)
- added REF**: MountingHole_2.2mm_M2_ISO14580, MountingHole:MountingHole_2.2mm_M2_ISO14580, B.Cu at (28.6, 152.8)
- added REF**: MountingHole_2.2mm_M2_ISO14580, MountingHole:MountingHole_2.2mm_M2_ISO14580, F.Cu at (195.6, 177.4)
- added REF**: MountingHole_2.2mm_M2_ISO14580, MountingHole:MountingHole_2.2mm_M2_ISO14580, F.Cu at (335.3, 152.8)
- added REF**: MountingHole_2.2mm_M2_ISO14580, MountingHole:MountingHole_2.2mm_M2_ISO14580, F.Cu at (335.3, 89.1)
- added REF**: MountingHole_2.2mm_M2_ISO14580, MountingHole:MountingHole_2.2mm_M2_ISO14580, B.Cu at (168.3, 177.4)
- added REF**: MountingHole_2.2mm_M2_ISO14580, MountingHole:MountingHole_2.2mm_M2_ISO14580, B.Cu at (95.3, 54.8)
- added REF**: MountingHole_2.2mm_M2_ISO14580, MountingHole:MountingHole_2.2mm_M2_ISO14580, B.Cu at (28.6, 89.1)
- added REF**: MountingHole_2.2mm_M2_ISO14580, MountingHole:MountingHole_2.2mm_M2_ISO14580, B.Cu at (161.9, 69.1)
- added REF**: MountingHole_2.2mm_M2_ISO14580, MountingHole:MountingHole_2.2mm_M2_ISO14580, B.Cu at (98.7, 165.1)
- added REF**: MountingHole_2.2mm_M2_ISO14580, MountingHole:MountingHole_2.2mm_M2_ISO14580, F.Cu at (268.6, 54.8)
- added REF**: MountingHole_2.2mm_M2_ISO14580, MountingHole:MountingHole_2.2mm_M2_ISO14580, F.Cu at (202.0, 69.1)
- added REF**: MountingHole_2.2mm_M2_ISO14580, MountingHole:MountingHole_2.2mm_M2_ISO14580, F.Cu at (265.2, 165.1)
- moved JL0 1.52 mm to (54.5, 73.9)
- moved JR0 1.52 mm to (309.4, 73.9)
Connections:
- JL1 pad 5: GND1 -> Net-(JL1-Pad5)
- JR1 pad 5: GND2 -> Net-(JR1-Pad5)
- RL0 pad 1: GND1 -> Net-(JL1-Pad5)
- RL1 pad 1: GND1 -> Net-(JL1-Pad5)
- RR0 pad 1: GND2 -> Net-(JR1-Pad5)
- RR1 pad 1: GND2 -> Net-(JR1-Pad5)
- USBL1 pad A1: GND1 -> Net-(JL1-Pad5)
- USBL1 pad A12: GND1 -> Net-(JL1-Pad5)
- USBL1 pad B1: GND1 -> Net-(JL1-Pad5)
- USBL1 pad B12: GND1 -> Net-(JL1-Pad5)
- USBL1 pad S1: GND1 -> Net-(JL1-Pad5)
- USBR0 pad A1: GND2 -> Net-(JR1-Pad5)
- USBR0 pad A12: GND2 -> Net-(JR1-Pad5)
- USBR0 pad B1: GND2 -> Net-(JR1-Pad5)
- USBR0 pad B12: GND2 -> Net-(JR1-Pad5)
- USBR0 pad S1: GND2 -> Net-(JR1-Pad5)
Routing:
- net GND1: track 886.5 -> 795.5 mm, vias 68 -> 65
- net Net-(JL1-Pad5): track 0.00 -> 89.5 mm
- net GND2: track 879.8 -> 794.4 mm
- net Net-(JR1-Pad5): track 0.00 -> 83.8 mm
- net R5V: track 821.1 -> 819.5 mm
- net Net-(JL0-Pad2): track 96.9 -> 95.4 mm
- net L5V: track 816.0 -> 814.5 mm
- net Net-(JR0-Pad2): track 102.1 -> 101.4 mm
- removed copper zone on B.Cu, net GND1
- removed copper zone on F.Cu, net GND1
- removed copper zone on B.Cu, net GND2
- removed copper zone on F.Cu, net GND2
Other:
- board size 316.6 x 144.6 mm -> 316.6 x 132.5 mm
